Commit message: modify logging typo, modify parameter to fit real experiments, tune a bit on control using realtime 1 and fast C3

File: examples/franka_trajectory_following/robot_properties_fingers/urdf/franka_box.urdf (robot description, URDF)
Before this commit: robot panda, 13 links, 12 joints
Links:
- link connection: geometry visual box size=0.3 0.3 0.0038
Joints:
- joint connection_to_box: origin xyz=0 0 -0.07450000000000001 -> xyz=0 0 -0.0538
